Commit message: Refine M6 Pro description: rear LiDAR, light-gray body, teleop limits
- Move LiDAR turret toward the rear (lidar_center_offset -0.13 m); the M6 Pro
  LiDAR is not centered. Also affects real-robot mapping (base_link->base_scan).
- Color the body/caster light gray (add light_gray material) to match the robot.
- Retune teleop_keyboard.yaml for wheel_track 0.233 m (old max_ang_vel 7.72 was
  derived from the Mini's track); values provisional pending physical calibration.

Co-Authored-By: Claude Opus 4.8 (1M context) <noreply@anthropic.com>

File: urdf/materials.xacro (robot description, xacro)
@@ -31,4 +31,7 @@
     <color rgba="1.0 1.0 1.0 1.0"/>
   </material>
+  <material name="light_gray">
+    <color rgba="0.8 0.8 0.8 1.0"/>
+  </material>
   <gazebo reference="wheel_left_link">
     <mu1>0.2</mu1>

File: urdf/params.xacro (robot description, xacro)
@@ -20,5 +20,9 @@
   <xacro:property name="laser_puck_diameter" value="0.070"/>
   <xacro:property name="laser_puck_offset" value="0.005"/>
-  <xacro:property name="lidar_center_offset" value="0.000"/>
+  <!-- LiDAR turret sits toward the REAR of the vacuum, not centered.
+       +X is forward, so a negative value shifts it back. Refine by measuring
+       the horizontal distance from the robot center to the LiDAR center and
+       setting this to its negative (meters). -->
+  <xacro:property name="lidar_center_offset" value="-0.13"/>
   <!-- N*m -->
   <xacro:property name="motor_stall_torque" value="0.5"/>

File: urdf/robot.urdf.xacro (robot description, xacro)
@@ -18,5 +18,5 @@
         <cylinder length="${lower_cylinder_height}" radius="${base_diameter/2}"/>
       </geometry>
-      <material name="white"/>
+      <material name="light_gray"/>
     </visual>
     <collision>
@@ -39,5 +39,5 @@
         <sphere radius="${caster_diameter/2}"/>
       </geometry>
-      <material name="white"/>
+      <material name="light_gray"/>
     </visual>
    <collision>

Commit message: Gray body color + front bumper contact sensors (sim)
- Color: body/caster light_gray (0.8, looked white) -> grey (0.5); drop light_gray.
- Bumpers: add left/right front bumper halves as NAMED collisions + visuals on
  base_link (named so the gz contact sensor references survive URDF->SDF without
  fixed-joint lumping). Add gz contact sensors + the Contact system in
  plugins.xacro, and bridge bumper_left/contact, bumper_right/contact to ROS
  (ros_gz_interfaces/msg/Contacts) in gz_bridge.yaml. Geometry is approximate -
  refine visually. The physical robot still uses /bumper (vacuum_ros2_bridge/Bumper).

Co-Authored-By: Claude Opus 4.8 (1M context) <noreply@anthropic.com>

File: urdf/materials.xacro (robot description, xacro)
@@ -31,7 +31,4 @@
     <color rgba="1.0 1.0 1.0 1.0"/>
   </material>
-  <material name="light_gray">
-    <color rgba="0.8 0.8 0.8 1.0"/>
-  </material>
   <gazebo reference="wheel_left_link">
     <mu1>0.2</mu1>

File: urdf/params.xacro (robot description, xacro)
@@ -35,4 +35,11 @@
   <xacro:property name="laser_puck_mass" value="0.150"/>
   <!-- ****************** **************** ****************** -->
+  <!-- Front bumpers (left/right halves), approximated as thin boxes hugging the
+       front perimeter. Geometry is a rough placeholder - refine visually in sim. -->
+  <xacro:property name="bumper_angle" value="35"/>    <!-- deg from front for each half -->
+  <xacro:property name="bumper_length" value="0.13"/> <!-- tangential -->
+  <xacro:property name="bumper_thickness" value="0.012"/> <!-- radial -->
+  <xacro:property name="bumper_height" value="0.045"/>
+  <xacro:property name="bumper_z" value="0.022"/>     <!-- center height in base_link frame -->
   <xacro:property name="DEG2RAD" value="0.0174533"/>
 </robot>

File: urdf/plugins.xacro (robot description, xacro)
@@ -27,4 +27,29 @@
       <joint_name>wheel_right_joint</joint_name>
     </plugin>
+    <!-- Processes the bumper contact sensors below. NOTE: the Contact system is
+         normally a WORLD-level system. If the bumper contact topics don't appear,
+         add this same plugin to the Gazebo world (kaiaai_gazebo living_room.world). -->
+    <plugin filename="gz-sim-contact-system" name="gz::sim::systems::Contact"/>
+  </gazebo>
+  <!-- Front bumper contact sensors. They watch the named bumper collisions on
+       base_link (see robot.urdf.xacro) and publish gz.msgs.Contacts, bridged to
+       ROS as ros_gz_interfaces/msg/Contacts (see config/gz_bridge.yaml). -->
+  <gazebo reference="base_link">
+    <sensor name="bumper_left" type="contact">
+      <always_on>true</always_on>
+      <update_rate>50</update_rate>
+      <contact>
+        <collision>bumper_left_collision</collision>
+      </contact>
+      <topic>bumper_left/contact</topic>
+    </sensor>
+    <sensor name="bumper_right" type="contact">
+      <always_on>true</always_on>
+      <update_rate>50</update_rate>
+      <contact>
+        <collision>bumper_right_collision</collision>
+      </contact>
+      <topic>bumper_right/contact</topic>
+    </sensor>
   </gazebo>
   <!-- gazebo reference="laser_frame" -->

File: urdf/robot.urdf.xacro (robot description, xacro)
@@ -6,4 +6,24 @@
   <xacro:include filename="materials.xacro" />
   <!-- ****************** **************** ****************** -->
+  <!-- Front bumper half as a thin box tangent to the body, placed on base_link
+       as a NAMED collision (so the Gazebo contact sensor can reference it
+       without fixed-joint lumping renaming it). 'angle' is degrees from front. -->
+  <xacro:macro name="front_bumper" params="name angle">
+    <visual>
+      <origin xyz="${(base_diameter/2)*cos(angle*DEG2RAD)} ${(base_diameter/2)*sin(angle*DEG2RAD)} ${bumper_z}"
+              rpy="0 0 ${(angle+90)*DEG2RAD}"/>
+      <geometry>
+        <box size="${bumper_length} ${bumper_thickness} ${bumper_height}"/>
+      </geometry>
+      <material name="dark"/>
+    </visual>
+    <collision name="${name}">
+      <origin xyz="${(base_diameter/2)*cos(angle*DEG2RAD)} ${(base_diameter/2)*sin(angle*DEG2RAD)} ${bumper_z}"
+              rpy="0 0 ${(angle+90)*DEG2RAD}"/>
+      <geometry>
+        <box size="${bumper_length} ${bumper_thickness} ${bumper_height}"/>
+      </geometry>
+    </collision>
+  </xacro:macro>
   <link name="base_footprint"/>
   <joint name="base_joint" type="fixed">
@@ -18,5 +38,5 @@
         <cylinder length="${lower_cylinder_height}" radius="${base_diameter/2}"/>
       </geometry>
-      <material name="light_gray"/>
+      <material name="grey"/>
     </visual>
     <collision>
@@ -26,4 +46,7 @@
       </geometry>
     </collision>
+    <!-- Front bumpers as named collisions on base_link (see macro above) -->
+    <xacro:front_bumper name="bumper_left_collision" angle="${bumper_angle}"/>
+    <xacro:front_bumper name="bumper_right_collision" angle="${-bumper_angle}"/>
     <xacro:solid_cylinder_inertia m="${lower_cylinder_mass}" r="${base_diameter/2}" h="${lower_cylinder_height}"/>
   </link>
@@ -39,5 +62,5 @@
         <sphere radius="${caster_diameter/2}"/>
       </geometry>
-      <material name="light_gray"/>
+      <material name="grey"/>
     </visual>
    <collision>
