Commit message: Retarget description package to Proscenic M6 Pro
Rename makerspet_mini -> proscenic_m6pro and adapt the Mini copy to the
Proscenic M6 Pro robot vacuum, which is bridged to ROS 2 via
remakeai/vacuum_ros2_bridge (SangamIO over TCP) instead of ESP32/micro-ROS.

- Rename package (package.xml, CMakeLists, kaiaai.yaml, URDF robot name)
- Re-dimension URDF to ~349mm dia / ~95mm tall / 0.233m wheel base; model as
  a flat cylinder + upright LiDAR turret; drop the domed head mesh and sdf/
- Un-flip the LiDAR frame (turret is upright, not an inverted LDS)
- Add launch/bringup.launch.py: bridge + robot_state_publisher + EKF
- Add config/ekf.yaml: robot_localization fuses /odom + /imu to publish the
  odom -> base_footprint TF the bridge omits and cartographer requires
- Rewrite README for the M6 Pro

Co-Authored-By: Claude Opus 4.8 (1M context) <noreply@anthropic.com>

File: urdf/params.xacro (robot description, xacro)
@@ -3,32 +3,30 @@
   <!-- ****************** ROBOT DIMENSIONS ****************** -->
   <!-- Units: meters, degrees, kg, N*m, m/s2 -->
-  <xacro:property name="wheel_diameter" value="0.043"/>
-  <xacro:property name="wheel_width" value="0.0055"/>
-  <xacro:property name="caster_diameter" value="0.017"/>
+  <!-- Proscenic M6 Pro: round body ~349mm dia, ~95mm tall (incl. LiDAR turret). -->
+  <!-- wheel_base 0.233m matches vacuum_ros2_bridge WHEEL_BASE used for odometry. -->
+  <!-- Values are approximate; refine against measurements of the physical robot. -->
+  <xacro:property name="wheel_diameter" value="0.065"/>
+  <xacro:property name="wheel_width" value="0.012"/>
+  <xacro:property name="caster_diameter" value="0.025"/>
   <!-- Caster center to base edge -->
-  <xacro:property name="caster_inset" value="0.011"/>
-  <xacro:property name="floor_clearance" value="0.0149"/>
-  <xacro:property name="base_diameter" value="0.124"/>
-  <xacro:property name="wheel_base" value="0.105043"/>
-  <xacro:property name="lower_cylinder_height" value="0.032"/>
-  <xacro:property name="laser_puck_height" value="0.016"/>
-  <xacro:property name="laser_puck_diameter" value="0.06"/>
-  <xacro:property name="laser_puck_offset" value="0.0384"/>
-  <xacro:property name="laser_motor_diameter" value="0.02"/>
-  <xacro:property name="lidar_motor_x_offset" value="0.04"/>
-  <xacro:property name="lidar_motor_z_offset" value="0.012"/>
-  <xacro:property name="laser_motor_height" value="0.01"/>
-  <xacro:property name="head_height" value="0.0388"/>
+  <xacro:property name="caster_inset" value="0.030"/>
+  <xacro:property name="floor_clearance" value="0.010"/>
+  <xacro:property name="base_diameter" value="0.349"/>
+  <xacro:property name="wheel_base" value="0.233"/>
+  <!-- Flat vacuum body height (LiDAR turret adds on top) -->
+  <xacro:property name="lower_cylinder_height" value="0.072"/>
+  <!-- LiDAR turret/puck on top of the body -->
+  <xacro:property name="laser_puck_height" value="0.018"/>
+  <xacro:property name="laser_puck_diameter" value="0.070"/>
+  <xacro:property name="laser_puck_offset" value="0.005"/>
   <xacro:property name="lidar_center_offset" value="0.000"/>
   <!-- N*m -->
-  <xacro:property name="motor_stall_torque" value="0.171616375"/>
+  <xacro:property name="motor_stall_torque" value="0.5"/>
   <xacro:property name="max_linear_acceleration" value="1"/>
-  <xacro:property name="lower_cylinder_mass" value="0.250"/>
+  <xacro:property name="lower_cylinder_mass" value="2.500"/>
   <!-- caster and battery weight -->
   <xacro:property name="caster_mass" value="0.050"/>
-  <xacro:property name="wheel_mass" value="0.050"/>
+  <xacro:property name="wheel_mass" value="0.100"/>
   <xacro:property name="laser_puck_mass" value="0.150"/>
-  <xacro:property name="laser_motor_mass" value="0.050"/>
-  <xacro:property name="head_mass" value="0.200"/>
   <!-- ****************** **************** ****************** -->
   <xacro:property name="DEG2RAD" value="0.0174533"/>

File: urdf/robot.urdf.xacro (robot description, xacro)
@@ -1,4 +1,4 @@
 <?xml version="1.0" ?>
-<robot name="makerspet_mini" xmlns:xacro="http://ros.org/wiki/xacro">
+<robot name="proscenic_m6pro" xmlns:xacro="http://ros.org/wiki/xacro">
   <xacro:include filename="params.xacro" />
   <xacro:include filename="inertial.xacro" />
@@ -101,8 +101,10 @@
     <xacro:solid_cylinder_inertia m="${wheel_mass}" r="${wheel_diameter/2}" h="${wheel_width}"/>
   </link>
+  <!-- Upright top-mounted LiDAR turret (+Z up, CCW scan) to match both the
+       Gazebo gpu_lidar sensor and the physical robot's vacuum_ros2_bridge /scan. -->
   <joint name="scan_joint" type="fixed">
     <parent link="base_link"/>
     <child link="base_scan"/>
-    <origin xyz="${lidar_center_offset} 0 ${lower_cylinder_height + laser_puck_offset}" rpy="0 -${pi} 0"/>
+    <origin xyz="${lidar_center_offset} 0 ${lower_cylinder_height + laser_puck_offset}" rpy="0 0 0"/>
   </joint>
   <link name="base_scan">
@@ -122,45 +124,3 @@
     <xacro:solid_cylinder_inertia m="${laser_puck_mass}" r="${laser_puck_diameter/2}" h="${laser_puck_height}"/>
   </link>
-  <joint name="scan_motor_joint" type="fixed">
-    <parent link="base_scan"/>
-    <child link="scan_motor"/>
-    <origin xyz="${lidar_motor_x_offset} 0 ${lidar_motor_z_offset}" rpy="0 -${pi} 0"/>
-  </joint>
-  <link name="scan_motor">
-    <visual>
-      <origin xyz="0 0 0" rpy="0 0 0"/>
-      <geometry>
-        <cylinder length="${laser_motor_height}" radius="${laser_motor_diameter/2}"/>
-      </geometry>
-      <material name="black"/>
-    </visual>
-    <collision>
-      <origin xyz="0 0 0" rpy="0 0 0"/>
-      <geometry>
-        <cylinder length="${laser_motor_height}" radius="${laser_motor_diameter/2}"/>
-      </geometry>
-    </collision>
-    <xacro:solid_cylinder_inertia m="${laser_motor_mass}" r="${laser_motor_diameter/2}" h="${laser_motor_height}"/>
-  </link>
-  <joint name="head_joint" type="fixed">
-    <parent link="base_link"/>
-    <child link="head_link"/>
-    <origin xyz="0 0 ${lower_cylinder_height}" rpy="0 0 0"/>
-  </joint>
-  <link name="head_link">
-    <visual>
-      <origin xyz="0 0 0" rpy="0 0 0"/>
-      <geometry>
-        <mesh filename="package://makerspet_mini/mesh/hemisphere.stl" scale="${0.001*base_diameter} ${0.001*base_diameter} ${0.001*head_height*2}"/>
-      </geometry>
-      <material name="red"/>
-    </visual>
-    <collision>
-      <origin xyz="0 0 ${head_height/2}" rpy="0 0 0"/>
-      <geometry>
-        <cylinder length="${head_height}" radius="${base_diameter/2}"/>
-      </geometry>
-    </collision>
-    <xacro:solid_semi_ellipsoid_inertia m="${head_mass}" x="${base_diameter/2}" y="${base_diameter/2}" z="${head_height}"/>
-  </link>
 </robot>

Commit message: Apply measured M6 Pro dimensions
From the physical robot:
- wheel_diameter 0.068 (68mm)
- wheel_base 0.235 (measured 235mm track)
- lidar_center_offset -0.0965 (LiDAR center 78mm in from rear edge)
- teleop max_ang_vel 2.55 (derived from 0.235m track)

Co-Authored-By: Claude Opus 4.8 (1M context) <noreply@anthropic.com>

File: urdf/params.xacro (robot description, xacro)
@@ -3,8 +3,8 @@
   <!-- ****************** ROBOT DIMENSIONS ****************** -->
   <!-- Units: meters, degrees, kg, N*m, m/s2 -->
-  <!-- Proscenic M6 Pro: round body ~349mm dia, ~95mm tall (incl. LiDAR turret). -->
-  <!-- wheel_base 0.233m matches vacuum_ros2_bridge WHEEL_BASE used for odometry. -->
-  <!-- Values are approximate; refine against measurements of the physical robot. -->
-  <xacro:property name="wheel_diameter" value="0.065"/>
+  <!-- Proscenic M6 Pro: round body 349mm dia (measured), ~95mm tall (incl. LiDAR turret). -->
+  <!-- wheel_base = measured wheel track 235mm. The bridge uses its own odometry
+       constant WHEEL_BASE = 0.233m (2mm less); negligible, calibrate empirically. -->
+  <xacro:property name="wheel_diameter" value="0.068"/>
   <xacro:property name="wheel_width" value="0.012"/>
   <xacro:property name="caster_diameter" value="0.025"/>
@@ -13,5 +13,5 @@
   <xacro:property name="floor_clearance" value="0.010"/>
   <xacro:property name="base_diameter" value="0.349"/>
-  <xacro:property name="wheel_base" value="0.233"/>
+  <xacro:property name="wheel_base" value="0.235"/>
   <!-- Flat vacuum body height (LiDAR turret adds on top) -->
   <xacro:property name="lower_cylinder_height" value="0.072"/>
@@ -21,8 +21,7 @@
   <xacro:property name="laser_puck_offset" value="0.005"/>
   <!-- LiDAR turret sits toward the REAR of the vacuum, not centered.
-       +X is forward, so a negative value shifts it back. Refine by measuring
-       the horizontal distance from the robot center to the LiDAR center and
-       setting this to its negative (meters). -->
-  <xacro:property name="lidar_center_offset" value="-0.13"/>
+       +X is forward, so negative shifts it back. Measured: LiDAR center is
+       78mm in from the rear edge -> 174.5mm radius - 78mm = 96.5mm behind center. -->
+  <xacro:property name="lidar_center_offset" value="-0.0965"/>
   <!-- N*m -->
   <xacro:property name="motor_stall_torque" value="0.5"/>

Commit message: Apply measured M6 Pro body and LiDAR housing dimensions
- lower_cylinder_height 0.079 (79mm body)
- laser_puck_height 0.018 (18mm LiDAR housing), seated flush (offset 0.009)
- laser_puck_diameter 0.083 (83mm)

Co-Authored-By: Claude Opus 4.8 (1M context) <noreply@anthropic.com>

File: urdf/params.xacro (robot description, xacro)
@@ -14,10 +14,11 @@
   <xacro:property name="base_diameter" value="0.349"/>
   <xacro:property name="wheel_base" value="0.235"/>
-  <!-- Flat vacuum body height (LiDAR turret adds on top) -->
-  <xacro:property name="lower_cylinder_height" value="0.072"/>
-  <!-- LiDAR turret/puck on top of the body -->
+  <!-- Flat vacuum body cylinder, measured 79mm tall (LiDAR housing on top) -->
+  <xacro:property name="lower_cylinder_height" value="0.079"/>
+  <!-- LiDAR housing, measured 18mm, seated flush on the body top -->
   <xacro:property name="laser_puck_height" value="0.018"/>
-  <xacro:property name="laser_puck_diameter" value="0.070"/>
-  <xacro:property name="laser_puck_offset" value="0.005"/>
+  <xacro:property name="laser_puck_diameter" value="0.083"/>
+  <!-- offset = laser_puck_height/2 so the housing bottom sits at the body top -->
+  <xacro:property name="laser_puck_offset" value="0.009"/>
   <!-- LiDAR turret sits toward the REAR of the vacuum, not centered.
        +X is forward, so negative shifts it back. Measured: LiDAR center is

Commit message: Correct floor clearance and body height
Floor gap measured ~12.5mm; the 79mm figure is the body top above the floor,
so the body cylinder itself is 66.5mm (79 - 12.5). LiDAR housing top ~97mm.

Co-Authored-By: Claude Opus 4.8 (1M context) <noreply@anthropic.com>

File: urdf/params.xacro (robot description, xacro)
@@ -11,9 +11,10 @@
   <!-- Caster center to base edge -->
   <xacro:property name="caster_inset" value="0.030"/>
-  <xacro:property name="floor_clearance" value="0.010"/>
+  <xacro:property name="floor_clearance" value="0.0125"/>
   <xacro:property name="base_diameter" value="0.349"/>
   <xacro:property name="wheel_base" value="0.235"/>
-  <!-- Flat vacuum body cylinder, measured 79mm tall (LiDAR housing on top) -->
-  <xacro:property name="lower_cylinder_height" value="0.079"/>
+  <!-- Body cylinder: top is 79mm above the floor, minus 12.5mm floor gap = 66.5mm tall.
+       LiDAR housing sits on top (body top 79mm + 18mm housing = ~97mm total height). -->
+  <xacro:property name="lower_cylinder_height" value="0.0665"/>
   <!-- LiDAR housing, measured 18mm, seated flush on the body top -->
   <xacro:property name="laser_puck_height" value="0.018"/>

Commit message: Bumper as continuous front-180 cylinder wall (faceted arc)
The two paddle bumpers left a gap at dead-center, so a head-on bump registered
no contact. Replace them with a continuous faceted arc that forms the front 180
deg of the body's cylindrical wall: left half 0..+90 deg, right half -90..0 deg,
6 facets each (overlapping, no gaps), meeting at the front. Facets are named
collisions on base_link and each contact sensor lists its half's facets. Facets
sit at the body radius and protrude ~5mm so they are the surface that touches
obstacles.

Co-Authored-By: Claude Opus 4.8 (1M context) <noreply@anthropic.com>

File: urdf/params.xacro (robot description, xacro)
@@ -35,11 +35,14 @@
   <xacro:property name="laser_puck_mass" value="0.150"/>
   <!-- ****************** **************** ****************** -->
-  <!-- Front bumpers (left/right halves), approximated as thin boxes hugging the
-       front perimeter. Geometry is a rough placeholder - refine visually in sim. -->
-  <xacro:property name="bumper_angle" value="35"/>    <!-- deg from front for each half -->
-  <xacro:property name="bumper_length" value="0.13"/> <!-- tangential -->
-  <xacro:property name="bumper_thickness" value="0.012"/> <!-- radial -->
-  <xacro:property name="bumper_height" value="0.045"/>
-  <xacro:property name="bumper_z" value="0.022"/>     <!-- center height in base_link frame -->
+  <!-- Front bumper = the front 180 deg of the body's cylindrical wall, modelled as
+       a continuous faceted arc. Left half spans 0..+90 deg, right half -90..0 deg
+       (they meet at the front, 0 deg, so there is no dead-center gap). Each half is
+       'bumper_facets_per_side' thin box facets, named so the contact sensors can
+       reference them; facets sit at the body radius and protrude a few mm so they
+       are the surface that touches obstacles. -->
+  <xacro:property name="bumper_facets_per_side" value="6"/>
+  <xacro:property name="bumper_thickness" value="0.010"/> <!-- radial; outer face ~5mm proud -->
+  <xacro:property name="bumper_height" value="0.050"/>
+  <xacro:property name="bumper_z" value="0.033"/>     <!-- center height in base_link frame -->
   <xacro:property name="DEG2RAD" value="0.0174533"/>
 </robot>

File: urdf/plugins.xacro (robot description, xacro)
@@ -32,7 +32,14 @@
     <plugin filename="gz-sim-contact-system" name="gz::sim::systems::Contact"/>
   </gazebo>
-  <!-- Front bumper contact sensors. They watch the named bumper collisions on
-       base_link (see robot.urdf.xacro) and publish gz.msgs.Contacts, bridged to
-       ROS as ros_gz_interfaces/msg/Contacts (see config/gz_bridge.yaml). -->
+  <!-- Lists all facet collision names for one bumper half, for the contact sensor. -->
+  <xacro:macro name="bumper_facet_collisions" params="prefix n i:=0">
+    <xacro:if value="${i &lt; n}">
+      <collision>${prefix}_${i}</collision>
+      <xacro:bumper_facet_collisions prefix="${prefix}" n="${n}" i="${i + 1}"/>
+    </xacro:if>
+  </xacro:macro>
+  <!-- Front bumper contact sensors. Each half watches all of its arc-facet
+       collisions on base_link (see robot.urdf.xacro) and publishes gz.msgs.Contacts,
+       bridged to ROS as ros_gz_interfaces/msg/Contacts (see config/gz_bridge.yaml). -->
   <gazebo reference="base_link">
     <sensor name="bumper_left" type="contact">
@@ -40,5 +47,5 @@
       <update_rate>50</update_rate>
       <contact>
-        <collision>bumper_left_collision</collision>
+        <xacro:bumper_facet_collisions prefix="bumper_left" n="${bumper_facets_per_side}"/>
       </contact>
       <topic>bumper_left/contact</topic>
@@ -48,5 +55,5 @@
       <update_rate>50</update_rate>
       <contact>
-        <collision>bumper_right_collision</collision>
+        <xacro:bumper_facet_collisions prefix="bumper_right" n="${bumper_facets_per_side}"/>
       </contact>
       <topic>bumper_right/contact</topic>

File: urdf/robot.urdf.xacro (robot description, xacro)
@@ -6,23 +6,32 @@
   <xacro:include filename="materials.xacro" />
   <!-- ****************** **************** ****************** -->
-  <!-- Front bumper half as a thin box tangent to the body, placed on base_link
-       as a NAMED collision (so the Gazebo contact sensor can reference it
-       without fixed-joint lumping renaming it). 'angle' is degrees from front. -->
-  <xacro:macro name="front_bumper" params="name angle">
+  <!-- One bumper facet: a thin box tangent to the body at angle 'ang' (deg from
+       front), at the body radius. Named collision so the contact sensor can list it. -->
+  <xacro:macro name="bumper_facet" params="prefix idx ang width">
     <visual>
-      <origin xyz="${(base_diameter/2)*cos(angle*DEG2RAD)} ${(base_diameter/2)*sin(angle*DEG2RAD)} ${bumper_z}"
-              rpy="0 0 ${(angle+90)*DEG2RAD}"/>
+      <origin xyz="${(base_diameter/2)*cos(ang*DEG2RAD)} ${(base_diameter/2)*sin(ang*DEG2RAD)} ${bumper_z}"
+              rpy="0 0 ${(ang+90)*DEG2RAD}"/>
       <geometry>
-        <box size="${bumper_length} ${bumper_thickness} ${bumper_height}"/>
+        <box size="${width} ${bumper_thickness} ${bumper_height}"/>
       </geometry>
       <material name="dark"/>
     </visual>
-    <collision name="${name}">
-      <origin xyz="${(base_diameter/2)*cos(angle*DEG2RAD)} ${(base_diameter/2)*sin(angle*DEG2RAD)} ${bumper_z}"
-              rpy="0 0 ${(angle+90)*DEG2RAD}"/>
+    <collision name="${prefix}_${idx}">
+      <origin xyz="${(base_diameter/2)*cos(ang*DEG2RAD)} ${(base_diameter/2)*sin(ang*DEG2RAD)} ${bumper_z}"
+              rpy="0 0 ${(ang+90)*DEG2RAD}"/>
       <geometry>
-        <box size="${bumper_length} ${bumper_thickness} ${bumper_height}"/>
+        <box size="${width} ${bumper_thickness} ${bumper_height}"/>
       </geometry>
     </collision>
+  </xacro:macro>
+  <!-- A 90-deg bumper half built from 'n' facets spanning a0 .. a0+90 deg.
+       Facet width = arc chord * 1.15 so neighbours overlap (continuous, no gaps). -->
+  <xacro:macro name="bumper_arc" params="prefix a0 n i:=0">
+    <xacro:if value="${i &lt; n}">
+      <xacro:bumper_facet prefix="${prefix}" idx="${i}"
+        ang="${a0 + (i + 0.5) * (90.0 / n)}"
+        width="${2 * (base_diameter/2) * sin(0.5 * (90.0/n) * DEG2RAD) * 1.15}"/>
+      <xacro:bumper_arc prefix="${prefix}" a0="${a0}" n="${n}" i="${i + 1}"/>
+    </xacro:if>
   </xacro:macro>
   <link name="base_footprint"/>
@@ -46,7 +55,8 @@
       </geometry>
     </collision>
-    <!-- Front bumpers as named collisions on base_link (see macro above) -->
-    <xacro:front_bumper name="bumper_left_collision" angle="${bumper_angle}"/>
-    <xacro:front_bumper name="bumper_right_collision" angle="${-bumper_angle}"/>
+    <!-- Continuous front bumper = front 180 deg of the cylinder wall (named
+         collisions on base_link). Left half 0..+90 deg, right half -90..0 deg. -->
+    <xacro:bumper_arc prefix="bumper_left" a0="0" n="${bumper_facets_per_side}"/>
+    <xacro:bumper_arc prefix="bumper_right" a0="-90" n="${bumper_facets_per_side}"/>
     <xacro:solid_cylinder_inertia m="${lower_cylinder_mass}" r="${base_diameter/2}" h="${lower_cylinder_height}"/>
   </link>
